File: akimbo.kicad_pcb (KiCad board)
At the start: 2 copper layers, 163.9 x 125.9 mm, 75 parts, among them J1 USB mini-B, J2 3.5mm TRRS, J3 3.5mm TRRS, K1 -, K11 -, K12 -, K13 -, K14 -, K15 -, K16 -, K17 -, K18 -, K19 -, K2 -, K20 -, K21 -, K22 -, K23 -, K24 -, K25 -, K26 -, K27 -, K28 -, K29 -, K3 -, K30 -, K4 -, K6 -, K7 -, K8 -, K9 -, U1 ATmega32U4, U2 MCP23017_SO, Y1 16M

Commit message: replace mcp23017 with pca9995
Parts:
- U2: value MCP23017_SO -> PCA9555D; footprint Package_SO:SOIC-28W_7.5x17.9mm_P1.27mm -> Package_SO:SOIC-24W_7.5x15.4mm_P1.27mm
- moved U2 1.26 mm to (53.4, 35.6), turned to 270 degrees
Connections:
- U2 pad 1: /row0 -> (no net)
- U2 pad 10: GND -> /col5
- U2 pad 11: (no net) -> /col0
- U2 pad 12: /sck -> GND
- U2 pad 13: /sda -> /row0
- U2 pad 14: (no net) -> /row1
- U2 pad 15: GND -> /row2
- U2 pad 16: GND -> /row3
- U2 pad 17: GND -> /row4
- U2 pad 18: +5V -> (no net)
- U2 pad 2: /row1 -> GND
- U2 pad 21: (no net) -> GND
- U2 pad 22: (no net) -> /sck
- U2 pad 23: /col3 -> /sda
- U2 pad 24: /col2 -> +5V
- U2 pad 3: /row2 -> GND
- U2 pad 4: /row3 -> (no net)
- U2 pad 5: /row4 -> (no net)
- U2 pad 6: (no net) -> /col3
- U2 pad 7: (no net) -> /col2
- U2 pad 8: (no net) -> /col1
- U2 pad 9: +5V -> /col4
Routing:
- net GND: track 80.9 -> 95.2 mm
- net +5V: track 85.6 -> 88.8 mm, vias 16 -> 17
- net /col4: track 169.6 -> 168.3 mm
- net /col3: track 189.1 -> 187.8 mm
- net /sda: track 159.5 -> 158.4 mm
- net /sck: track 162.5 -> 161.4 mm
- net /col0: track 101.3 -> 100.2 mm
- net /col5: track 173.7 -> 172.6 mm
