File: akimbo.sch (KiCad schematic (older format))
At the start: 75 parts, among them J1 USB-C, J2 3.5mm TRRS, J3 3.5mm TRRS, K1 -, K11 -, K12 -, K13 -, K14 -, K15 -, K16 -, K17 -, K18 -, K19 -, K2 -, K20 -, K21 -, K22 -, K23 -, K24 -, K25 -, K26 -, K27 -, K28 -, K29 -, K3 -, K30 -, K4 -, K6 -, K7 -, K8 -, K9 -, U1 ATmega32U4, U2 MCP23017_SO, Y1 16M

Commit message: schematic cleanup, BOM essentially complete
Parts:
- K2, K3, K4: footprint akimbo:SW_Cherry_MX_1.25u_PCB_Reversible -> akimbo:SW_Cherry_MX_1.00u_PCB_Reversible
Other:
- note added: "I/O EXPANDER - RIGHT HALF"
- note added: "KEY MATRIX - BOTH HALVES"
- note added: "MICROCONTROLLER - LEFT HALF"
- note added: "SUGGESTED LAYOUT"
- moved on the sheet: C1, C2, C3, H1, H2, H3, H4, J1, J2, J3, K1, R1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

Commit message: decoupling caps; better crystal-μC routing
Parts:
- added C4: 10u, Capacitor_SMD:C_0805_2012Metric_Pad1.15x1.40mm_HandSolder, symbol Device:C_Small
- added C5: 10n, Capacitor_SMD:C_0805_2012Metric_Pad1.15x1.40mm_HandSolder, symbol Device:C_Small
Connections:
- net +5V: now also C4.2, C5.1
- net GND: now also C4.1, C5.2
Other:
- note added: "Decoupling\nPlace near U1/U2 footprint"
Changed lines of the file:
@@
 	1375 3400 1375 3700
 Wire Wire Line
-	2675 3000 2675 2300
+	2675 3000 2675 2475
 Connection ~ 2675 3000
 Wire Wire Line
@@
 Connection ~ 2325 2600
 Wire Wire Line
-	2325 2600 2325 2200
+	2325 2600 2325 2475
 Wire Wire Line
 	1775 3100 1725 3100
@@
 	1    0    0    1
 $EndComp
+$Comp
+L Device:C_Small C4
+U 1 1 5D6A5286
+P 2500 2475
+F 0 "C4" V 2450 2375 50  0000 C CNN
+F 1 "10u" V 2450 2575 50  0000 C CNN
+F 2 "Capacitor_SMD:C_0805_2012Metric_Pad1.15x1.40mm_HandSolder" H 2500 2475 50  0001 C CNN
+F 3 "~" H 2500 2475 50  0001 C CNN
+	1    2500 2475
+	0    1    1    0
+$EndComp
+Wire Wire Line
+	2400 2475 2325 2475
+Connection ~ 2325 2475
+Wire Wire Line
+	2325 2475 2325 2200
+Wire Wire Line
+	2600 2475 2675 2475
+Connection ~ 2675 2475
+Wire Wire Line
+	2675 2475 2675 2300
+$Comp
+L power:+5V #PWR019
+U 1 1 5D6E3942
+P 5250 6975
+F 0 "#PWR019" H 5250 6825 50  0001 C CNN
+F 1 "+5V" H 5250 7115 50  0000 C CNN
+F 2 "" H 5250 6975 50  0001 C CNN
+F 3 "" H 5250 6975 50  0001 C CNN
+	1    5250 6975
+	1    0    0    -1
+$EndComp
+$Comp
+L power:GND #PWR020
+U 1 1 5D6E3EFD
+P 5250 7525
+F 0 "#PWR020" H 5250 7275 50  0001 C CNN
+F 1 "GND" H 5250 7375 50  0000 C CNN
+F 2 "" H 5250 7525 50  0001 C CNN
+F 3 "" H 5250 7525 50  0001 C CNN
+	1    5250 7525
+	1    0    0    -1
+$EndComp
+$Comp
+L Device:C_Small C5
+U 1 1 5D6E44E7
+P 5250 7250
+F 0 "C5" H 5260 7320 50  0000 L CNN
+F 1 "10n" H 5260 7170 50  0000 L CNN
+F 2 "Capacitor_SMD:C_0805_2012Metric_Pad1.15x1.40mm_HandSolder" H 5250 7250 50  0001 C CNN
+F 3 "~" H 5250 7250 50  0001 C CNN
+	1    5250 7250
+	1    0    0    -1
+$EndComp
+Wire Wire Line
+	5250 6975 5250 7150
+Wire Wire Line
+	5250 7350 5250 7525
+Text Notes 5500 7325 0    50   ~ 0
+Decoupling\nPlace near U1/U2 footprint
 $EndSCHEMATC

Commit message: minor tweaks, no functional changes
Other:
- note removed: "2019-08-28"
Changed lines of the file:
@@
 Wire Wire Line
 	3325 3300 3325 3200
-Text Notes 11825 10400 0    250  Italic 50
+Text Notes 11950 10400 0    250  Italic 50
 AKIMBO!
 Wire Notes Line width 48 style solid
-	11825 10450 13275 10450
-Text Notes 13395 10400 0    75   ~ 0
+	11950 10450 13400 10450
+Text Notes 13520 10400 0    75   ~ 0
 PROTOTYPE
-Text Notes 12960 11070 0    50   ~ 0
-2019-08-28
-Text Notes 11995 10670 0    50   ~ 0
-1
-Text Notes 12105 10670 0    50   ~ 0
-1
-Text Notes 14365 10070 0    50   Italic 0
-© 2019 Rachel K
-Text Notes 14365 10160 0    50   ~ 0
-https://github.com/rkanati/akimbo.git
 Wire Notes Line style solid rgb(132, 0, 0)
 	14325 9960 14325 10570
@@
 Text Notes 5500 7325 0    50   ~ 0
 Decoupling\nPlace near U1/U2 footprint
+Text Notes 14365 10160 0    50   ~ 0
+https://github.com/rkanati/akimbo.git
+Text Notes 14365 10070 0    50   Italic 0
+© 2019 Rachel K
 $EndSCHEMATC
